Commit message: Update s-model_articulated_macro.xacro
Fixed joints

File: robotiq_s_model_visualization/cfg/s-model_articulated_macro.xacro (robot description, xacro)
@@ -38,5 +38,5 @@
 		<!-- joint list -->
 		<!-- WARNING: LIMITS NOT CORRECT -->
-		<joint name="${prefix}palm_finger_1_joint" type="revolute">
+		<joint name="${prefix}palm_finger_1_joint" type="fixed">
 			<parent link="${prefix}palm"/>
 			<child link="${prefix}finger_1_link_0"/>
@@ -46,5 +46,5 @@
 		</joint>
 		<!-- WARNING: LIMITS NOT CORRECT -->
-		<joint name="${prefix}palm_finger_2_joint" type="revolute">
+		<joint name="${prefix}palm_finger_2_joint" type="fixed">
 			<parent link="${prefix}palm"/>
 			<child link="${prefix}finger_2_link_0"/>
