Commit message: Update s-model_finger_articulated_macro.xacro
Fixed joints

File: robotiq_s_model_visualization/cfg/s-model_finger_articulated_macro.xacro (robot description, xacro)
@@ -104,5 +104,5 @@
 		<!-- joint list -->
 		<!-- WARNING: LIMITS NOT CORRECT -->
-		<joint name="${prefix}joint_1" type="revolute">
+		<joint name="${prefix}joint_1" type="fixed">
 			<parent link="${prefix}link_0"/>
 			<child link="${prefix}link_1"/>
@@ -112,5 +112,5 @@
 		</joint>
 		<!-- WARNING: LIMITS NOT CORRECT -->
-		<joint name="${prefix}joint_2" type="revolute">
+		<joint name="${prefix}joint_2" type="fixed">
 			<parent link="${prefix}link_1"/>
 			<child link="${prefix}link_2"/>
@@ -120,5 +120,5 @@
 		</joint>
 		<!-- WARNING: LIMITS NOT CORRECT -->
-		<joint name="${prefix}joint_3" type="revolute">
+		<joint name="${prefix}joint_3" type="fixed">
 			<parent link="${prefix}link_2"/>
 			<child link="${prefix}link_3"/>
